File: KICAD/SAMD21G_TrainingBoard.kicad_pcb (KiCad board)
At the start: 2 copper layers, 100 x 100 mm, 65 parts, among them CN1 CN-PICkit4_ARM, CN2 USB_Mini_B, CN3 UART-FTDI-TTL-232R-3V3, CN4 USB_A, CN5 CN-POWER, IC1 SAMD21G18A, IC2 NJM2391DL1-33, IC3 GT20L16J1Y, SW1 SW_PUSH_2, SW2 SW_PUSH_2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

Commit message: amend USB Type A connector Power Supply
Connections:
- CN1 pad 4: (no net) -> Net-(CN1-Pad4)
- CN1 pad 6: (no net) -> Net-(CN1-Pad6)
- CN1 pad 7: (no net) -> Net-(CN1-Pad7)
- CN2 pad 4: (no net) -> Net-(CN2-Pad4)
- CN3 pad 3: (no net) -> Net-(CN3-Pad3)
- CN4 pad 1: Net-(CN2-Pad1) -> Net-(C17-Pad2)
- CN4 pad 5: (no net) -> Net-(CN4-Pad5)
- CN4 pad 6: (no net) -> Net-(CN4-Pad6)
- IC1 pad 19: (no net) -> Net-(IC1-Pad19)
- IC1 pad 39: (no net) -> Net-(IC1-Pad39)
- IC1 pad 4: (no net) -> Net-(IC1-Pad4)
- IC1 pad 41: (no net) -> Net-(IC1-Pad41)
- LCD1 pad 6: (no net) -> Net-(LCD1-Pad6)
- LCD1 pad 7: (no net) -> Net-(LCD1-Pad7)
- LCD1 pad 8: (no net) -> Net-(LCD1-Pad8)
- PAD1 pad 1: (no net) -> Net-(PAD1-Pad1)
- PAD2 pad 1: (no net) -> Net-(PAD2-Pad1)
- PAD3 pad 1: (no net) -> Net-(PAD3-Pad1)
- PAD4 pad 1: (no net) -> Net-(PAD4-Pad1)
- SDCARD1 pad 1: (no net) -> Net-(SDCARD1-Pad1)
- SDCARD1 pad 10: (no net) -> Net-(SDCARD1-Pad10)
- SDCARD1 pad 8: (no net) -> Net-(SDCARD1-Pad8)
- SDCARD1 pad 9: (no net) -> Net-(SDCARD1-Pad9)
- SE1 pad 3: (no net) -> Net-(SE1-Pad3)
Routing:
- net Net-(CN2-Pad1): track 40.4 -> 6.79 mm
- net Net-(C17-Pad2): track 15.2 -> 48.4 mm, vias 0 -> 1
- net Net-(CN2-Pad2): track 44.0 -> 43.3 mm
